File: morph00/morph00.kicad_sch (KiCad schematic)
At the start: 0 parts

Commit message: Changed some stuff
Parts:
- added C1, C2: C, Capacitor_THT:C_Disc_D5.0mm_W2.5mm_P2.50mm, symbol Device:C
- added R1, R2, R3, R4: Resistor, Resistor_THT:R_Axial_DIN0207_L6.3mm_D2.5mm_P7.62mm_Horizontal, symbol ScottoKeebs:Placeholder_Resistor
- added SW1, SW2, SW3, SW4, SW5, SW6: SW_Push, symbol Switch:SW_Push
- added SW7: RotaryEncoder_Switch, symbol Device:RotaryEncoder_Switch
- added U1: (no value), ScottoKeebs_MCU:Adafruit_KB2040, symbol ScottoKeebs:MCU_Adafruit_KB2040
Connections:
- new net: R1.1, R3.1, SW7.A
- new net: R2.2, R4.1, SW7.B
- new net +3.3V: R1.2, R2.1, U1.18 (VCC)
- new net GND: C1.2, C2.2, SW1.1, SW2.1, SW3.1, SW4.1, SW5.1, SW6.1, SW7.C, SW7.S2, U1.5 (GND)
- new net Key Switch 1: SW1.2, U1.6 (2/PD1)
- new net Key Switch 2: SW2.2, U1.7 (3/PD0)
- new net Key Switch 3: SW3.2, U1.8 (4/PD4)
- new net Key Switch 4: SW4.2, U1.9 (5/PC6)
- new net Key Switch 5: SW5.2, U1.10 (6/PD7)
- new net Key Switch 6: SW6.2, U1.11 (7/PE6)
- new net Rotary Encoder A: C1.1, R3.2, U1.12 (8/PB4)
- new net Rotary Encoder B: C2.1, R4.2, U1.13 (9/PB5)
- new net Rotary Encoder Push Button Switch: SW7.S1, U1.19 (A3/PF4)

Commit message: tt
Parts:
- removed SW7: RotaryEncoder_Switch, symbol Device:RotaryEncoder_Switch
- added DS1: (no value), OLED:TZT_5.5_OLED_SSD1322, symbol OLED:TZT_5.5_OLED_SSD1322
- added SW8: Rotary Encoder Switch, Rotary_Encoder:RotaryEncoder_Alps_EC11E-Switch_Vertical_H20mm, symbol Device:RotaryEncoder_Switch_MP
- SW1, SW2, SW3, SW4, SW5, SW6: footprint (none) -> Button_Switch_Keyboard:SW_Cherry_MX_1.00u_PCB
Connections:
- net +3.3V: now also DS1.2 (VCC)
- net GND: now also DS1.1 (GND), SW8.C, SW8.MP, SW8.S2
- net Rotary Encoder Push Button Switch: now also U1.26 (10/PB6), SW8.S1; no longer U1.19 (A3/PF4)
- net at R1.1, R3.1: now also SW8.A
- net at R2.2, R4.1: now also SW8.B
- net OLED Data: now reaches U1.20 (A2/PF5)
- net OLED Data: now also DS1.4 (SDA(Data))
- net OLED Reset: now reaches U1.21 (A1/PF6)
- net OLED Reset: now also DS1.5 (RST(Reset))
- net OLED DC: now reaches U1.22 (A0/PF7)
- net OLED DC: now also DS1.6 (DC)
- net OLED CS: now reaches U1.23 (15/PB1)
- net OLED CS: now also DS1.7 (CS)
- new net OLED Clock: DS1.3 (SCL(Clock)), U1.19 (A3/PF4)
- no-connect marks 0 -> 11
