File: morph00/morph00.kicad_pcb (KiCad board)
At the start: 2 copper layers, 222.5 x 97.5 mm, 19 parts, among them SW1 SW_Push, SW2 SW_Push, SW3 SW_Push, SW4 SW_Push, SW5 SW_Push, SW6 SW_Push, SW8 Rotary Encoder Switch

Commit message: code and pcb changes and docs
Routing:
- net GND: track 334.4 -> 336.4 mm
- net +3.3V: track 288.7 -> 290.0 mm
- net /Rotary Encoder A: track 214.9 -> 213.6 mm
- added copper zone on B.Cu, net GND
- added copper zone on F.Cu, net GND
