File: hardware/kicad_files/morph00/morph00.kicad_pcb (KiCad board)
At the start: 2 copper layers, 222.5 x 97.5 mm, 19 parts, among them SW1 SW_Push, SW2 SW_Push, SW3 SW_Push, SW4 SW_Push, SW5 SW_Push, SW6 SW_Push, SW8 Rotary Encoder Switch

Commit message: Uodate for final submission
Routing:
- net /OLED DC: track 53.4 -> 51.6 mm
- net /OLED Clock: track 70.8 -> 69.3 mm
- net +3.3V: track 337.1 -> 336.1 mm
- net /OLED Data: track 64.4 -> 63.5 mm
- net /OLED Reset: track 58.8 -> 57.9 mm
- net /OLED CS: track 47.0 -> 46.4 mm
